File: KiCAD_Files/VANGUARD-PASIL/VANGUARD-PASIL.kicad_sch (KiCad schematic)
At the start: 17 parts, among them J1 U_MX1508_FRONT, J2 U_MX1508_REAR, J3 Conn_01x04, J4 Conn_01x04, J6 NRF24L01+PA+LNA(2.4 GHz), M1 M_FR, M2 M_FL, M3 M_RL, M4 M_RR, U1 BlackPill_STM32F411CEU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

Commit message: Bugs Squashed and Documentation updated!
Connections:
- net TIM3_CH1_PWM(IN1) renamed TIM3_CH2_PWM(IN1)
